Commit message: test sim

File: warehouse_rb1_files/rb1_ros2/rb1_ros2_description/urdf/elevator/elevator.gazebo.xacro (robot description, xacro)
@@ -8,5 +8,5 @@
 			<kd value="1.0" />
 			<fdir1 value="1 0 0"/>
-			<material>Gazebo/Black</material>
+			<!--material>Gazebo/Black</material-->
 			<turnGravityOff>false</turnGravityOff>
 			<!--kp>500000.0</kp>

File: warehouse_rb1_files/rb1_ros2/rb1_ros2_description/urdf/elevator/elevator.urdf.xacro (robot description, xacro)
@@ -77,5 +77,5 @@
 		</inertial>
 		<visual>
-			<origin xyz="0 0 0" rpy="0 0 0" />
+			<origin xyz="0 0 0" rpy="-${pi/2} 0 0" />
 			<xacro:if value="${hq}">
 				<geometry>
@@ -93,5 +93,5 @@
 		</visual>
 		<collision>
-			<origin xyz="0 0 0" rpy="0 0 0 " />
+			<origin xyz="0 0 0" rpy="-${pi/2} 0 0 " />
 			<mass>2</mass>
 			<geometry>
