Commit message: Se elimino la collision de la flecha

File: warehouse_rb1_files/rb1_ros2/rb1_ros2_description/urdf/elevator/elevator.urdf.xacro (robot description, xacro)
@@ -92,5 +92,5 @@
 			</material>
 		</visual>
-		<collision>
+		<!--collision>
 			<origin xyz="0 0 0" rpy="-${pi/2} 0 0 " />
 			<mass>2</mass>
@@ -98,5 +98,5 @@
 				<mesh filename="package://rb1_ros2_description/meshes/elevator/rb1_elevator_platform.dae"/>
 			</geometry>
-		</collision>
+		</collision-->
 	</link>
 	<xacro:elevator_gazebo prefix="${prefix}" />
